Commit message: [MISC] Genesis fabric test

File: genesis/assets/urdf/DG3F/urdf/delto_gripper_3f.urdf (robot description, URDF)
Before this commit: robot delto_gripper_3f, 17 links, 16 joints
Links:
- added link tip1_force_frame
- added link tip2_force_frame
- added link tip3_force_frame
Joints:
- added joint tip1_force_frame_joint: type fixed, parent F1_TIP, child tip1_force_frame, origin xyz=0.045 0.0 0.0 rpy=0 0 0
- added joint tip2_force_frame_joint: type fixed, parent F2_TIP, child tip2_force_frame, origin xyz=0.045 0.0 0.0 rpy=0 0 0
- added joint tip3_force_frame_joint: type fixed, parent F3_TIP, child tip3_force_frame, origin xyz=0.045 0.0 0.0 rpy=0 0 0
